Commit message: change links to point to correct meshes in new hyq repo

File: urdf_files/HyQ/hyq.urdf (robot description, URDF)
Before this commit: robot hyq, 18 links, 17 joints
Links:
- link trunk: geometry collision mesh filename=package://hyq_description/meshes/leg/trunk.dae scale=1 1 1; visual mesh filename=package://hyq_description/meshes/leg/trunk.dae scale=1 1 1
